File: hardware/turret-pdb/logic/turret-logic.kicad_pcb (KiCad board)
At the start: 2 copper layers, 70 x 58 mm, 14 parts, among them J12 Stack link, J5 ESC left, J6 ESC right, J7 TTLinker, J8 TFmini Plus, J9 Light gate, U1 Freenove ESP32-S3 WROOM, U2 Adafruit 757

Commit message: Route the power board
Co-Authored-By: Claude Opus 5.5 <noreply@anthropic.com>
Parts:
- moved J12 25.2 mm to (77.1, 97.0)
- moved H3 10.0 mm to (44.0, 104.0)
- moved H4 10.0 mm to (106.0, 104.0)
- moved J5 10.0 mm to (96.0, 81.0)
- moved J6 10.0 mm to (101.0, 81.0)
- moved J7 10.0 mm to (44.0, 82.0)
- moved J8 10.0 mm to (96.0, 93.5)
- moved J9 10.0 mm to (101.0, 93.5)
- moved R3 10.0 mm to (106.0, 98.0)
- moved R4 10.0 mm to (106.0, 82.0)
- moved U1 10.0 mm to (89.8, 100.5)
- moved U2 10.0 mm to (59.5, 60.5)
Other:
- board size 70 x 58 mm -> 70 x 68 mm
Changed lines of the file:
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@@
 	(footprint "turret-logic:Freenove_ESP32-S3_WROOM_Socket"
 		(layer "F.Cu")
-		(at 89.8 90.5 90)
+		(at 89.8 100.5 90)
 		(descr "Freenove ESP32-S3 WROOM in two 1x20 female strips; pull the contacts marked x, holes only on used pins")
 		(property "Reference" "U1"
@@
 	(footprint "turret-logic:Adafruit_757_UpsideDown"
 		(layer "F.Cu")
-		(at 59.5 50.5 270)
+		(at 59.5 60.5 270)
 		(descr "Adafruit 757 4-channel BSS138 level shifter, mounted components down")
 		(property "Reference" "U2"
@@
 	(footprint "turret-logic:PinHeader_1x03_P2.54mm_ESC"
 		(layer "F.Cu")
-		(at 96 71 90)
+		(at 96 81 90)
 		(descr "1x3 2.54 mm male header, pads on the solder side only")
 		(property "Reference" "J5"
@@
 	(footprint "turret-logic:PinHeader_1x03_P2.54mm_ESC"
 		(layer "F.Cu")
-		(at 101 71 90)
+		(at 101 81 90)
 		(descr "1x3 2.54 mm male header, pads on the solder side only")
 		(property "Reference" "J6"
@@
 	(footprint "turret-logic:PinHeader_1x04_P2.54mm"
 		(layer "F.Cu")
-		(at 44 72 270)
+		(at 44 82 270)
 		(descr "1x4 2.54 mm male header, pads on the solder side only")
 		(property "Reference" "J7"
@@
 	(footprint "turret-logic:PinHeader_1x04_P2.54mm"
 		(layer "F.Cu")
-		(at 96 83.5 90)
+		(at 96 93.5 90)
 		(descr "1x4 2.54 mm male header, pads on the solder side only")
 		(property "Reference" "J8"
@@
 	(footprint "turret-logic:PinHeader_1x03_P2.54mm"
 		(layer "F.Cu")
-		(at 101 83.5 90)
+		(at 101 93.5 90)
 		(descr "1x3 2.54 mm male header, pads on the solder side only")
 		(property "Reference" "J9"
@@
 	(footprint "turret-logic:R_Axial_P10.16mm_Horizontal"
 		(layer "F.Cu")
-		(at 106 88 90)
+		(at 106 98 90)
 		(descr "Axial resistor, 0207, 10.16 mm lead spacing")
 		(property "Reference" "R3"
@@
 	(footprint "turret-logic:R_Axial_P10.16mm_Horizontal"
 		(layer "F.Cu")
-		(at 106 72 90)
+		(at 106 82 90)
 		(descr "Axial resistor, 0207, 10.16 mm lead spacing")
 		(property "Reference" "R4"
@@
 	(footprint "turret-logic:WirePads_1x05_NoTie"
 		(layer "F.Cu")
-		(at 52 95 90)
+		(at 77.1 97 90)
 		(descr "Solder holes for stranded wire, zip-tie holes at both ends for strain relief")
 		(property "Reference" "J12"
@@
 	(footprint "turret-logic:MountingHole_M3"
 		(layer "F.Cu")
-		(at 44 94)
+		(at 44 104)
 		(descr "M3 mounting hole, no copper")
 		(property "Reference" "H3"
@@
 	(footprint "turret-logic:MountingHole_M3"
 		(layer "F.Cu")
-		(at 106 94)
+		(at 106 104)
 		(descr "M3 mounting hole, no copper")
 		(property "Reference" "H4"
@@
 	(gr_line
 		(start 110 44)
-		(end 110 94)
+		(end 110 104)
 		(stroke
 			(width 0.1)
@@
 	)
 	(gr_line
-		(start 106 98)
-		(end 44 98)
+		(start 106 108)
+		(end 44 108)
 		(stroke
 			(width 0.1)
@@
 	)
 	(gr_line
-		(start 40 94)
+		(start 40 104)
 		(end 40 44)
 		(stroke
@@
 	)
 	(gr_arc
-		(start 110 94)
-		(mid 108.8284 96.8284)
-		(end 106 98)
+		(start 110 104)
+		(mid 108.8284 106.8284)
+		(end 106 108)
 		(stroke
 			(width 0.1)
@@
 	)
 	(gr_arc
-		(start 44 98)
-		(mid 41.1716 96.8284)
-		(end 40 94)
+		(start 44 108)
+		(mid 41.1716 106.8284)
+		(end 40 104)
 		(stroke
 			(width 0.1)

Commit message: Route the logic board
Co-Authored-By: Claude Opus 5.5 <noreply@anthropic.com>
Parts:
- moved J7 60.4 mm to (101.0, 62.0), turned to 90 degrees
- moved R3 60.2 mm to (48.5, 80.2), turned to 270 degrees
- moved R4 54.0 mm to (52.0, 80.2), turned to 270 degrees
- moved J9 51.6 mm to (49.5, 96.0), turned to 0 degrees
- moved U2 24.4 mm to (83.5, 64.7), turned to 180 degrees
- moved J6 5.90 mm to (101.1, 75.1), turned to 180 degrees
- moved J5 5.15 mm to (101.1, 80.2), turned to 180 degrees
- moved J8 2.44 mm to (97.5, 95.4)
Connections:
- U2 pad A1: PUSH_SIG_3V3 -> BUS_TX_3V3
- U2 pad A2: BUS_RX_3V3 -> PUSH_SIG_3V3
- U2 pad A4: BUS_TX_3V3 -> BUS_RX_3V3
- U2 pad B1: PUSH_SIG -> BUS_TX
- U2 pad B2: BUS_RX -> PUSH_SIG
- U2 pad B4: BUS_TX -> BUS_RX
Routing:
- net GND: track 0.00 -> 171.2 mm, vias 0 -> 5
- net +5V: track 0.00 -> 91.7 mm, vias 0 -> 2
- net +3V3: track 0.00 -> 85.6 mm, vias 0 -> 3
- net BUS_RX: track 0.00 -> 41.4 mm
- net PUSH_SIG: track 0.00 -> 31.3 mm, vias 0 -> 2
- net PUSH_SIG_3V3: track 0.00 -> 26.1 mm
- net BUS_TX: track 0.00 -> 22.7 mm
- net ARM_SENSE: track 0.00 -> 22.2 mm, vias 0 -> 2
- net GATE: track 0.00 -> 18.1 mm
- net VBAT_SENSE: track 0.00 -> 13.4 mm
- net BUS_TX_3V3: track 0.00 -> 10.8 mm
- net GATE_LED: track 0.00 -> 8.89 mm
- net BUS_RX_3V3: track 0.00 -> 8.20 mm
- net TF_RX: track 0.00 -> 4.96 mm
- net ESC_R: track 0.00 -> 4.91 mm
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